File: board/dron-ze-smietnika/dron-ze-smietnika.kicad_sch (KiCad schematic)
At the start: 0 parts

Commit message: MPU6050 doesnt want to work
Parts:
- added C1, C2, C3, C4, C5, C6: C, symbol Device:C
- added R1, R2, R3: R, symbol Device:R
- added U1: STM8S005K6T6C, STM8S005K6T6C:QFP80P900X900X160-32N, symbol MCU_STM8S005:STM8S005K6T6C
- added U2: MPU-6050, Sensor_Motion:InvenSense_QFN-24_4x4mm_P0.5mm, symbol Sensor_Motion:MPU-6050
Connections:
- new net: C2.1, U2.20 (CPOUT)
- new net: C3.1, U2.10 (REGOUT)
- new net: C5.2, C6.1, U1.5 (VCAP)
- new net: C6.2, U1.6 (VDD), U1.7 (VDDIO)
- new net: R3.2, U1.1 (~{RST})
- new net: C5.1, U1.4 (VSS)
- new net +3.3V: C1.1, R1.1, R2.1, R3.1, U2.13 (VDD)
- new net GND: C1.2, C2.2, C3.2, C4.2, U2.1 (CLKIN), U2.11 (FSYNC), U2.18 (GND), U2.9 (AD0)
- new net SCL: R1.2, U1.12 (PB4/I2C_SCL/AIN4), U2.23 (SCL)
- new net SDA: R2.2, U1.11 (PB5/I2C_SDA/AIN5), U2.24 (SDA)
- new net V_LOGIC: C4.1, U2.8 (VLOGIC)
- no-connect marks 0 -> 3
